Commit message: updated a little

File: body.urdf (robot description, URDF)
Before this commit: robot robot, 3 links, 2 joints
Links:
- removed link LeftLeg
- removed link RightLeg
- removed link Torso
- added link Link0, mass 1; collision box size=0.7473530819385881 0.3281331689191723 1.3635767806290302; visual box size=0.7473530819385881 0.3281331689191723 1.3635767806290302
- added link Link1, mass 1; collision box size=1.7257484094688824 0.2499374618338066 1.5245427102808593; visual box size=1.7257484094688824 0.2499374618338066 1.5245427102808593
- added link Link2, mass 1; collision box size=1.867682050806843 1.459411868197388 1.8685619002088933; visual box size=1.867682050806843 1.459411868197388 1.8685619002088933
- added link Link3, mass 1; collision box size=1.5715716386265786 1.7346931362743436 1.8515897517586104; visual box size=1.5715716386265786 1.7346931362743436 1.8515897517586104
- added link Link4, mass 1; collision box size=0.20301609901613368 0.9847417979273321 0.2328073068605297; visual box size=0.20301609901613368 0.9847417979273321 0.2328073068605297
- added link Link5, mass 1; collision box size=1.8452492613653853 0.7325331532239012 0.634579426699905; visual box size=1.8452492613653853 0.7325331532239012 0.634579426699905
- added link Link6, mass 1; collision box size=0.34851665363217854 0.3993896021495803 1.2461452026079378; visual box size=0.34851665363217854 0.3993896021495803 1.2461452026079378
- added link Link7, mass 1; collision box size=1.5144308897534355 1.9119361520945084 0.44859069419211084; visual box size=1.5144308897534355 1.9119361520945084 0.44859069419211084
- added link Start, mass 1; collision box size=1 1 1; visual box size=1 1 1
Joints:
- removed joint Torso_LeftLeg
- removed joint Torso_RightLeg
- added joint Link0_Link1: type revolute, parent Link0, child Link1, origin xyz=0.37367654096929404 0.16406658445958616 0.6817883903145151 rpy=0 0 0, axis 1 0 0, limit lower=-3.14159 upper=3.14159 effort=0.0 velocity=0.0
- added joint Link1_Link2: type revolute, parent Link1, child Link2, origin xyz=0.8628742047344412 0.1249687309169033 0.7622713551404297 rpy=0 0 0, axis 1 0 0, limit lower=-3.14159 upper=3.14159 effort=0.0 velocity=0.0
- added joint Link2_Link3: type revolute, parent Link2, child Link3, origin xyz=0.9338410254034215 0.729705934098694 0.9342809501044467 rpy=0 0 0, axis 1 0 0, limit lower=-3.14159 upper=3.14159 effort=0.0 velocity=0.0
- added joint Link3_Link4: type revolute, parent Link3, child Link4, origin xyz=0.7857858193132893 0.8673465681371718 0.9257948758793052 rpy=0 0 0, axis 1 0 0, limit lower=-3.14159 upper=3.14159 effort=0.0 velocity=0.0
- added joint Link4_Link5: type revolute, parent Link4, child Link5, origin xyz=0.10150804950806684 0.49237089896366604 0.11640365343026485 rpy=0 0 0, axis 1 0 0, limit lower=-3.14159 upper=3.14159 effort=0.0 velocity=0.0
- added joint Link5_Link6: type revolute, parent Link5, child Link6, origin xyz=0.9226246306826926 0.3662665766119506 0.3172897133499525 rpy=0 0 0, axis 1 0 0, limit lower=-3.14159 upper=3.14159 effort=0.0 velocity=0.0
- added joint Link6_Link7: type revolute, parent Link6, child Link7, origin xyz=0.17425832681608927 0.19969480107479015 0.6230726013039689 rpy=0 0 0, axis 1 0 0, limit lower=-3.14159 upper=3.14159 effort=0.0 velocity=0.0
- added joint Start_Link0: type revolute, parent Start, child Link0, origin xyz=0.5 0 0 rpy=0 0 0, axis 1 0 0, limit lower=-3.14159 upper=3.14159 effort=0.0 velocity=0.0

Commit message: done

File: body.urdf (robot description, URDF)
Before this commit: robot robot, 9 links, 8 joints
Links:
- added link Link8, mass 1; collision box size=0.27201478713254035 0.5002503363640718 0.5299083344548569; visual box size=0.27201478713254035 0.5002503363640718 0.5299083344548569
- link Link0: geometry collision box size=1.0676430640180345 0.3159017647202928 1.0490340270961227; visual box size=1.0676430640180345 0.3159017647202928 1.0490340270961227
- link Link1: geometry collision box size=1.1519244192842975 0.22542307070188025 1.573403288857272; visual box size=1.1519244192842975 0.22542307070188025 1.573403288857272
- link Link2: geometry collision box size=1.332492940598871 0.6303090116989801 1.7471103793738045; visual box size=1.332492940598871 0.6303090116989801 1.7471103793738045
- link Link3: geometry collision box size=1.7408433291827368 1.0067316119647445 0.8393586854573145; visual box size=1.7408433291827368 1.0067316119647445 0.8393586854573145
- link Link4: geometry collision box size=1.2205308786066904 1.1013493909224592 1.973210445552139; visual box size=1.2205308786066904 1.1013493909224592 1.973210445552139
- link Link5: geometry collision box size=0.8056600548770101 0.7153237374892194 1.2381169133055208; visual box size=0.8056600548770101 0.7153237374892194 1.2381169133055208
- link Link6: geometry collision box size=0.3845551600758318 0.8958386387943784 1.5152940174858653; visual box size=0.3845551600758318 0.8958386387943784 1.5152940174858653
- link Link7: geometry collision box size=0.7826246401843087 1.9580521735967784 1.9042547227137452; visual box size=0.7826246401843087 1.9580521735967784 1.9042547227137452
Joints:
- added joint Link7_Link8: type revolute, parent Link7, child Link8, origin xyz=0.7826246401843087 0 0 rpy=0 0 0, axis 1 0 0, limit lower=-3.14159 upper=3.14159 effort=0.0 velocity=0.0
- joint Link0_Link1: origin xyz=0.37367654096929404 0.16406658445958616 0.6817883903145151 rpy=0 0 0 -> xyz=1.0676430640180345 0 0 rpy=0 0 0
- joint Link1_Link2: origin xyz=0.8628742047344412 0.1249687309169033 0.7622713551404297 rpy=0 0 0 -> xyz=1.1519244192842975 0 0 rpy=0 0 0
- joint Link2_Link3: origin xyz=0.9338410254034215 0.729705934098694 0.9342809501044467 rpy=0 0 0 -> xyz=1.332492940598871 0 0 rpy=0 0 0
- joint Link3_Link4: origin xyz=0.7857858193132893 0.8673465681371718 0.9257948758793052 rpy=0 0 0 -> xyz=1.7408433291827368 0 0 rpy=0 0 0
- joint Link4_Link5: origin xyz=0.10150804950806684 0.49237089896366604 0.11640365343026485 rpy=0 0 0 -> xyz=1.2205308786066904 0 0 rpy=0 0 0
- joint Link5_Link6: origin xyz=0.9226246306826926 0.3662665766119506 0.3172897133499525 rpy=0 0 0 -> xyz=0.8056600548770101 0 0 rpy=0 0 0
- joint Link6_Link7: origin xyz=0.17425832681608927 0.19969480107479015 0.6230726013039689 rpy=0 0 0 -> xyz=0.3845551600758318 0 0 rpy=0 0 0

Commit message: updated for assignment 7

File: body.urdf (robot description, URDF)
Before this commit: robot robot, 10 links, 9 joints
Links:
- removed link Link5
- removed link Link6
- removed link Link7
- removed link Link8
- link Link0: geometry collision box size=1.3522836435536805 0.7020100655028527 1.8779538411356655; visual box size=1.3522836435536805 0.7020100655028527 1.8779538411356655
- link Link1: geometry collision box size=1.25755213154533 1.3520501386095465 1.0865469026877672; visual box size=1.25755213154533 1.3520501386095465 1.0865469026877672
- link Link2: geometry collision box size=0.7068087661990952 1.6659620741558119 1.29016888932811; visual box size=0.7068087661990952 1.6659620741558119 1.29016888932811
- link Link3: geometry collision box size=1.9809394259725293 0.5235508826385595 0.7454209549057358; visual box size=1.9809394259725293 0.5235508826385595 0.7454209549057358
- link Link4: geometry collision box size=0.21435040420542323 1.5043385163451006 1.899087850715868; visual box size=0.21435040420542323 1.5043385163451006 1.899087850715868
Joints:
- removed joint Link0_Link1
- removed joint Link1_Link2
- removed joint Link2_Link3
- removed joint Link3_Link4
- removed joint Link4_Link5
- removed joint Link5_Link6
- removed joint Link6_Link7
- removed joint Link7_Link8
- added joint Link0_Link3: type revolute, parent Link0, child Link3, origin xyz=0.6761418217768402 0 -0.9389769205678328 rpy=0 0 0, axis 1 0 0, limit lower=-3.14159 upper=3.14159 effort=0.0 velocity=0.0
- added joint Start_Link1: type revolute, parent Start, child Link1, origin xyz=0.5 0 0 rpy=0 0 0, axis 1 0 0, limit lower=-3.14159 upper=3.14159 effort=0.0 velocity=0.0
- added joint Start_Link2: type revolute, parent Start, child Link2, origin xyz=-0.5 0 0 rpy=0 0 0, axis 1 0 0, limit lower=-3.14159 upper=3.14159 effort=0.0 velocity=0.0
- added joint Start_Link4: type revolute, parent Start, child Link4, origin xyz=0 0 0.5 rpy=0 0 0, axis 0 0 1, limit lower=-3.14159 upper=3.14159 effort=0.0 velocity=0.0
- joint Start_Link0: axis 1 0 0 -> 0 0 1; origin xyz=0.5 0 0 rpy=0 0 0 -> xyz=0 0 -0.5 rpy=0 0 0
