Commit message: updated

File: 1.urdf (robot description, URDF)
Before this commit: robot robot, 8 links, 7 joints
Links:
- removed link Link7
- added link Link3, mass 1; collision box size=1.8855930562390273 0.4670063051161376 0.4505472436327163; visual box size=1.8855930562390273 0.4670063051161376 0.4505472436327163
- link Link1: geometry collision box size=1.7076403561926312 1.2016177807743802 1.356129853278402; visual box size=1.7076403561926312 1.2016177807743802 1.356129853278402
- link Link2: geometry collision box size=1.9865781419169173 1.7479037518315217 0.41760192765045157; visual box size=1.9865781419169173 1.7479037518315217 0.41760192765045157
- link Link4: geometry collision box size=0.7460633196792517 1.257645091058407 1.788462201497344; visual box size=0.7460633196792517 1.257645091058407 1.788462201497344
- link Link5: geometry collision box size=1.735918310747642 1.0644085514316852 1.538715179527757; visual box size=1.735918310747642 1.0644085514316852 1.538715179527757
- link Link8: geometry collision box size=0.8669407999623442 1.5189784560593584 0.9003603775432492; visual box size=0.8669407999623442 1.5189784560593584 0.9003603775432492
- link Link9: geometry collision box size=1.6516772594040279 1.177265803788609 1.6730301956030909; visual box size=1.6516772594040279 1.177265803788609 1.6730301956030909
Joints:
- removed joint Link1_Link4
- removed joint Link1_Link9
- removed joint Link2_Link8
- removed joint Link4_Link5
- removed joint Link5_Link7
- removed joint Start_Link2
- added joint Link1_Link2: type revolute, parent Link1, child Link2, origin xyz=0 0 -1.356129853278402 rpy=0 0 0, axis 0 0 1, limit lower=-3.14159 upper=3.14159 effort=0.0 velocity=0.0
- added joint Link2_Link3: type revolute, parent Link2, child Link3, origin xyz=-0.9932890709584586 0 -0.20880096382522578 rpy=0 0 0, axis 1 0 0, limit lower=-3.14159 upper=3.14159 effort=0.0 velocity=0.0
- added joint Link3_Link4: type revolute, parent Link3, child Link4, origin xyz=-0.9427965281195136 0 -0.8470321239468943 rpy=0 0 0, axis 0 0 1, limit lower=-3.14159 upper=3.14159 effort=0.0 velocity=0.0
- added joint Link3_Link5: type revolute, parent Link3, child Link5, origin xyz=-0.9427965281195136 0 0.8470321239468943 rpy=0 0 0, axis 0 0 1, limit lower=-3.14159 upper=3.14159 effort=0.0 velocity=0.0
- added joint Link4_Link8: type revolute, parent Link4, child Link8, origin xyz=0 0 -1.788462201497344 rpy=0 0 0, axis 0 0 1, limit lower=-3.14159 upper=3.14159 effort=0.0 velocity=0.0
- added joint Link8_Link9: type revolute, parent Link8, child Link9, origin xyz=0 0.7594892280296792 -0.5223881269927215 rpy=0 0 0, axis 0 1 0, limit lower=-3.14159 upper=3.14159 effort=0.0 velocity=0.0
- joint Start_Link1: axis 0 1 0 -> 0 0 1; origin xyz=0 0.5 0 rpy=0 0 0 -> xyz=0 0 -0.5 rpy=0 0 0
