Commit message: updated readme

File: 0.urdf (robot description, URDF)
Before this commit: robot robot, 9 links, 8 joints
Links:
- removed link Link3
- added link Link10, mass 1; collision box size=0.6105934541197509 0.6317357071511767 0.43523937245860767; visual box size=0.6105934541197509 0.6317357071511767 0.43523937245860767
- added link Link5, mass 1; collision box size=1.7164284016523284 1.816711618444182 1.3904236239649548; visual box size=1.7164284016523284 1.816711618444182 1.3904236239649548
- link Link1: geometry collision box size=1.7746353893443885 1.2857341303304894 1.793376438743545; visual box size=1.7746353893443885 1.2857341303304894 1.793376438743545
- link Link2: geometry collision box size=0.7957554941416414 0.8928220627507888 1.4529003016711277; visual box size=0.7957554941416414 0.8928220627507888 1.4529003016711277
- link Link4: geometry collision box size=1.0577557856168853 0.3616838501520686 1.5636870595395862; visual box size=1.0577557856168853 0.3616838501520686 1.5636870595395862
- link Link6: geometry collision box size=0.5455010208885124 0.40702232059049825 1.4462291939113583; visual box size=0.5455010208885124 0.40702232059049825 1.4462291939113583
- link Link7: geometry collision box size=0.5782422113692858 1.653884425257418 1.9816574331961991; visual box size=0.5782422113692858 1.653884425257418 1.9816574331961991
- link Link8: geometry collision box size=0.7582461415281785 1.31966205162576 0.5765349883271609; visual box size=0.7582461415281785 1.31966205162576 0.5765349883271609
- link Link9: geometry collision box size=0.38399014139984117 1.6328010150330379 0.2643645817319974; visual box size=0.38399014139984117 1.6328010150330379 0.2643645817319974
- link Start: geometry collision box size=0.6346406391332584 1.0013162301904162 1.6793172844484376; visual box size=0.6346406391332584 1.0013162301904162 1.6793172844484376
Joints:
- removed joint Link1_Link6
- removed joint Link1_Link8
- removed joint Link4_Link7
- removed joint Link8_Link9
- removed joint Start_Link2
- removed joint Start_Link3
- added joint Link1_Link2: type revolute, parent Link1, child Link2, origin xyz=0.9674546913764208 0.6428670651652447 0 rpy=0 0 0, axis 0 1 0, limit lower=-3.14159 upper=3.14159 effort=0.0 velocity=0.0
- added joint Link4_Link10: type revolute, parent Link4, child Link10, origin xyz=0.5288778928084427 0 -0.7818435297697931 rpy=0 0 0, axis 0 0 1, limit lower=-3.14159 upper=3.14159 effort=0.0 velocity=0.0
- added joint Link4_Link5: type revolute, parent Link4, child Link5, origin xyz=0.5288778928084427 0 0.7818435297697931 rpy=0 0 0, axis 0 0 1, limit lower=-3.14159 upper=3.14159 effort=0.0 velocity=0.0
- added joint Link4_Link9: type revolute, parent Link4, child Link9, origin xyz=0.5288778928084427 0.1808419250760343 0 rpy=0 0 0, axis 0 1 0, limit lower=-3.14159 upper=3.14159 effort=0.0 velocity=0.0
- added joint Link5_Link6: type revolute, parent Link5, child Link6, origin xyz=0.8582142008261642 0 0.9307741958381591 rpy=0 0 0, axis 1 0 0, limit lower=-3.14159 upper=3.14159 effort=0.0 velocity=0.0
- added joint Link5_Link8: type revolute, parent Link5, child Link8, origin xyz=0 0 1.8615483916763182 rpy=0 0 0, axis 0 0 1, limit lower=-3.14159 upper=3.14159 effort=0.0 velocity=0.0
- added joint Start_Link7: type revolute, parent Start, child Link7, origin xyz=0 0 -0.5 rpy=0 0 0, axis 0 0 1, limit lower=-3.14159 upper=3.14159 effort=0.0 velocity=0.0
- joint Link1_Link4: origin xyz=-1.106545709377797 0 0 rpy=0 0 0 -> xyz=1.9349093827528416 0 0 rpy=0 0 0
- joint Start_Link1: origin xyz=-0.5 0 0 rpy=0 0 0 -> xyz=0.5 0 0 rpy=0 0 0

File: 3.urdf (robot description, URDF)
Before this commit: robot robot, 10 links, 9 joints
Links:
- removed link Link3
- removed link Link4
- removed link Link5
- removed link Link9
- added link Link10, mass 1; collision box size=0.6038972875126074 0.968777930980703 1.3856870419704619; visual box size=0.6038972875126074 0.968777930980703 1.3856870419704619
- added link Link11, mass 1; collision box size=0.5357270977576166 1.1826641878162292 1.7085336621636489; visual box size=0.5357270977576166 1.1826641878162292 1.7085336621636489
- added link Link12, mass 1; collision box size=0.4792620115917124 0.8879053723284391 0.6755992701621509; visual box size=0.4792620115917124 0.8879053723284391 0.6755992701621509
- added link Link13, mass 1; collision box size=0.7530870264645366 1.9817676867498186 1.4877764622739762; visual box size=0.7530870264645366 1.9817676867498186 1.4877764622739762
- link Link1: geometry collision box size=0.2831327365661206 0.2896999502416703 1.7756136756055507; visual box size=0.2831327365661206 0.2896999502416703 1.7756136756055507
- link Link2: geometry collision box size=1.9105202559338643 0.2505311640088768 0.2322652745332563; visual box size=1.9105202559338643 0.2505311640088768 0.2322652745332563
- link Link6: geometry collision box size=1.5826764978327563 1.4456003590043063 1.1994368751868998; visual box size=1.5826764978327563 1.4456003590043063 1.1994368751868998
- link Link7: geometry collision box size=1.9971853263390322 0.2848538164610074 0.9317237736251649; visual box size=1.9971853263390322 0.2848538164610074 0.9317237736251649
- link Link8: geometry collision box size=0.4334971164334714 1.435055979635569 1.861873651147745; visual box size=0.4334971164334714 1.435055979635569 1.861873651147745
- link Start: geometry collision box size=1.6364185776577171 0.9699425513242794 1; visual box size=1.6364185776577171 0.9699425513242794 1
Joints:
- removed joint Link1_Link3
- removed joint Link1_Link5
- removed joint Link1_Link7
- removed joint Link2_Link4
- removed joint Link3_Link6
- removed joint Link4_Link8
- removed joint Link4_Link9
- added joint Link10_Link12: type revolute, parent Link10, child Link12, origin xyz=0 -0.4843889654903515 0.7444536448718051 rpy=0 0 0, axis 0 1 0, limit lower=-3.14159 upper=3.14159 effort=0.0 velocity=0.0
- added joint Link10_Link13: type revolute, parent Link10, child Link13, origin xyz=0 0 1.4889072897436102 rpy=0 0 0, axis 0 0 1, limit lower=-3.14159 upper=3.14159 effort=0.0 velocity=0.0
- added joint Link1_Link8: type revolute, parent Link1, child Link8, origin xyz=0 0 -1.069063320416559 rpy=0 0 0, axis 0 0 1, limit lower=-3.14159 upper=3.14159 effort=0.0 velocity=0.0
- added joint Link2_Link6: type revolute, parent Link2, child Link6, origin xyz=0.9552601279669322 0 0.11613263726662815 rpy=0 0 0, axis 1 0 0, limit lower=-3.14159 upper=3.14159 effort=0.0 velocity=0.0
- added joint Link6_Link7: type revolute, parent Link6, child Link7, origin xyz=1.4405653450867841 0 0 rpy=0 0 0, axis 1 0 0, limit lower=-3.14159 upper=3.14159 effort=0.0 velocity=0.0
- added joint Link7_Link10: type revolute, parent Link7, child Link10, origin xyz=0.9985926631695161 0 0.46586188681258245 rpy=0 0 0, axis 0 0 1, limit lower=-3.14159 upper=3.14159 effort=0.0 velocity=0.0
- added joint Link7_Link11: type revolute, parent Link7, child Link11, origin xyz=0.9985926631695161 0.1424269082305037 0 rpy=0 0 0, axis 0 1 0, limit lower=-3.14159 upper=3.14159 effort=0.0 velocity=0.0
- joint Start_Link1: axis 1 0 0 -> 0 0 1; origin xyz=0.5 0 0 rpy=0 0 0 -> xyz=0 0 -0.5 rpy=0 0 0
- joint Start_Link2: axis 0 1 0 -> 0 0 1; origin xyz=0 -0.5 0 rpy=0 0 0 -> xyz=0 0 0.5 rpy=0 0 0

File: 4.urdf (robot description, URDF)
Before this commit: robot robot, 10 links, 9 joints
Links:
- removed link Link9
- link Link1: geometry collision box size=0.8760162531614937 0.6353518991907352 0.9391204795650361; visual box size=0.8760162531614937 0.6353518991907352 0.9391204795650361
- link Link2: geometry collision box size=0.95819773076701 0.98680882561835 1.3829004874443531; visual box size=0.95819773076701 0.98680882561835 1.3829004874443531
- link Link3: geometry collision box size=1.993590536095618 1.471624697485628 1.8582131835104905; visual box size=1.993590536095618 1.471624697485628 1.8582131835104905
- link Link4: geometry collision box size=1.5705909832760687 0.9781745532390533 1.114034592809385; visual box size=1.5705909832760687 0.9781745532390533 1.114034592809385
- link Link5: geometry collision box size=0.3882665464414199 0.9706856321371817 0.393435949821914; visual box size=0.3882665464414199 0.9706856321371817 0.393435949821914
- link Link6: geometry collision box size=0.3791331900300262 1.7579807439256812 1.8133581648591177; visual box size=0.3791331900300262 1.7579807439256812 1.8133581648591177
- link Link7: geometry collision box size=1.3642186180669087 1.5499334661614725 1.9262627210565832; visual box size=1.3642186180669087 1.5499334661614725 1.9262627210565832
- link Link8: geometry collision box size=1.4886731034106473 0.6621261440051518 0.22880211330657257; visual box size=1.4886731034106473 0.6621261440051518 0.22880211330657257
- link Start: geometry collision box size=1 0.7755555202687354 1.4542073176366395; visual box size=1 0.7755555202687354 1.4542073176366395
Joints:
- removed joint Link1_Link2
- removed joint Link1_Link7
- removed joint Link3_Link4
- removed joint Link3_Link5
- removed joint Link5_Link6
- removed joint Link8_Link9
- added joint Link1_Link6: type revolute, parent Link1, child Link6, origin xyz=-0.5299857667207379 0 -0.46956023978251804 rpy=0 0 0, axis 0 0 1, limit lower=-3.14159 upper=3.14159 effort=0.0 velocity=0.0
- added joint Link2_Link4: type revolute, parent Link2, child Link4, origin xyz=0.479098865383505 0 0.9003703749556335 rpy=0 0 0, axis 1 0 0, limit lower=-3.14159 upper=3.14159 effort=0.0 velocity=0.0
- added joint Link4_Link5: type revolute, parent Link4, child Link5, origin xyz=0.9537280772548464 0 -0.5570172964046926 rpy=0 0 0, axis 0 0 1, limit lower=-3.14159 upper=3.14159 effort=0.0 velocity=0.0
- added joint Link4_Link7: type revolute, parent Link4, child Link7, origin xyz=0.9537280772548464 -0.48908727661952667 0 rpy=0 0 0, axis 0 1 0, limit lower=-3.14159 upper=3.14159 effort=0.0 velocity=0.0
- added joint Start_Link2: type revolute, parent Start, child Link2, origin xyz=0 0 0.5 rpy=0 0 0, axis 0 0 1, limit lower=-3.14159 upper=3.14159 effort=0.0 velocity=0.0
- joint Link2_Link3: axis 1 0 0 -> 0 1 0; origin xyz=-0.9932890709584586 0 -0.20880096382522578 rpy=0 0 0 -> xyz=0 -0.32372737663009826 0.9003703749556335 rpy=0 0 0
- joint Link4_Link8: axis 0 0 1 -> 0 1 0; origin xyz=0 0 -1.788462201497344 rpy=0 0 0 -> xyz=0.9537280772548464 0.48908727661952667 0 rpy=0 0 0
- joint Start_Link1: axis 0 0 1 -> 1 0 0; origin xyz=0 0 -0.5 rpy=0 0 0 -> xyz=-0.5 0 0 rpy=0 0 0

File: 7.urdf (robot description, URDF)
Before this commit: robot robot, 8 links, 7 joints
Links:
- removed link Link8
- removed link Link9
- added link Link2, mass 1; collision box size=1.961536125478573 1.5485578897629 1.2197361155647841; visual box size=1.961536125478573 1.5485578897629 1.2197361155647841
- added link Link4, mass 1; collision box size=1.2961067624956535 1.1403079001557022 1.9077679323772625; visual box size=1.2961067624956535 1.1403079001557022 1.9077679323772625
- link Link1: geometry collision box size=0.24309541587240888 1.9520484530180366 1.792565670266386; visual box size=0.24309541587240888 1.9520484530180366 1.792565670266386
- link Link3: geometry collision box size=0.5341841893479514 0.48658991683335984 1.8411355331686885; visual box size=0.5341841893479514 0.48658991683335984 1.8411355331686885
- link Link5: geometry collision box size=1.9491492673268527 1.0248114764208087 0.667224032411865; visual box size=1.9491492673268527 1.0248114764208087 0.667224032411865
- link Link6: geometry collision box size=1.8651730307905388 0.29460192083657444 1.8994289234513033; visual box size=1.8651730307905388 0.29460192083657444 1.8994289234513033
- link Link7: geometry collision box size=1.900671058138932 1.0485692391791863 0.5563196856475787; visual box size=1.900671058138932 1.0485692391791863 0.5563196856475787
- link Start: geometry collision box size=0.29306678180163304 0.2886333283398708 0.6840854932353673; visual box size=0.29306678180163304 0.2886333283398708 0.6840854932353673
Joints:
- removed joint Link1_Link3
- removed joint Link1_Link8
- removed joint Link6_Link7
- removed joint Link6_Link9
- removed joint Start_Link6
- added joint Link1_Link2: type revolute, parent Link1, child Link2, origin xyz=0 -0.9760242265090183 -0.645523913658748 rpy=0 0 0, axis 0 1 0, limit lower=-3.14159 upper=3.14159 effort=0.0 velocity=0.0
- added joint Link3_Link4: type revolute, parent Link3, child Link4, origin xyz=0.2670920946739757 0 0.9205677665843442 rpy=0 0 0, axis 0 0 1, limit lower=-3.14159 upper=3.14159 effort=0.0 velocity=0.0
- added joint Link3_Link6: type revolute, parent Link3, child Link6, origin xyz=0.5341841893479514 0 0 rpy=0 0 0, axis 1 0 0, limit lower=-3.14159 upper=3.14159 effort=0.0 velocity=0.0
- added joint Link4_Link7: type revolute, parent Link4, child Link7, origin xyz=0 0 1.9077679323772625 rpy=0 0 0, axis 0 0 1, limit lower=-3.14159 upper=3.14159 effort=0.0 velocity=0.0
- added joint Start_Link3: type revolute, parent Start, child Link3, origin xyz=0.5 0 0 rpy=0 0 0, axis 1 0 0, limit lower=-3.14159 upper=3.14159 effort=0.0 velocity=0.0
- joint Link3_Link5: origin xyz=-0.9526473144658512 0 -0.8870213865907469 rpy=0 0 0 -> xyz=0.2670920946739757 0 -0.9205677665843442 rpy=0 0 0
